File: Kicad/EMM/MZ-2000_EMM.kicad_pcb (KiCad board)
At the start: 2 copper layers, 115.8 x 142.7 mm, 44 parts, among them J1 Conn_02x22_Row_Letter_First, U1 74LS04, U10 74LS193, U11 74LS138, U12 74LS138, U13 HM628512LFP-5, U14 74LS11, U15 74LS245, U2 74LS04, U3 74LS14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

Commit message: Add files via upload
Parts:
- added D3: 1S4, Diode_THT:D_DO-41_SOD81_P10.16mm_Horizontal, F.Cu at (76.1, 175.7)
- added R3: 10k, Resistor_THT:R_Axial_DIN0207_L6.3mm_D2.5mm_P7.62mm_Horizontal, F.Cu at (68.5, 168.1)
- added S3: SLIDE_SWITCH_3P, Connector_PinHeader_2.54mm:PinHeader_1x03_P2.54mm_Vertical, F.Cu at (88.8, 196.0)
Connections:
- U11 pad 4: Net-(R2-Pad2) -> Net-(U11-Pad4)
- U11 pad 5: Net-(R2-Pad2) -> Net-(U11-Pad4)
- U12 pad 4: Net-(R2-Pad2) -> Net-(U11-Pad4)
- U12 pad 5: Net-(R2-Pad2) -> Net-(U11-Pad4)
- U13 pad 29: /x3_WR -> Net-(R3-Pad2)
- U2 pad 10: (no net) -> Net-(U2-Pad10)
- U2 pad 11: GND -> /x3_WR
- U2 pad 3: GND -> Net-(U11-Pad4)
- U2 pad 4: (no net) -> Net-(U2-Pad4)
- U2 pad 5: GND -> Net-(U2-Pad4)
- U2 pad 6: (no net) -> Net-(R2-Pad2)
- U2 pad 8: (no net) -> Net-(D3-Pad2)
- U2 pad 9: GND -> Net-(U2-Pad10)
- U5 pad 8: Net-(R2-Pad2) -> Net-(U11-Pad4)
Routing:
- net Net-(D3-Pad2): track 0.00 -> 102.2 mm
- net Net-(U11-Pad4): track 0.00 -> 88.5 mm
- net Net-(R3-Pad2): track 0.00 -> 50.3 mm
- net Net-(D3-Pad1): track 0.00 -> 25.6 mm
- net GND: track 611.6 -> 593.4 mm, vias 1 -> 2
- net /A2: track 71.6 -> 55.3 mm
- net /x3_WR: track 83.6 -> 99.8 mm, vias 0 -> 1
- net Net-(U8-Pad12): track 60.1 -> 44.3 mm
- net +5V: track 448.5 -> 463.7 mm
- net Net-(U4-Pad6): track 54.4 -> 41.1 mm
- net Net-(R2-Pad2): track 147.3 -> 134.3 mm
- net Net-(U13-Pad23): track 68.5 -> 81.5 mm, vias 2 -> 0
- net Net-(U13-Pad7): track 33.9 -> 44.8 mm
- net Net-(U10-Pad5): track 51.6 -> 60.9 mm
- net /D2: track 117.7 -> 126.5 mm, vias 0 -> 1
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Other:
- board text added: "EMM for MZ-2000 Rev1.2"
- board text added: "RAM"
- board text added: "ROM"
- board text removed: "EMM for MZ-2000"

Commit message: Add files via upload
Parts:
- D1, D2: value 1S4 -> 1N4148
Other:
- board text added: "1N4148"

Commit message: Add files via upload
Parts:
- removed D3: 1S4, Diode_THT:D_DO-41_SOD81_P10.16mm_Horizontal
- added Q1: 2N7000, Package_TO_SOT_THT:TO-92, F.Cu at (48.8, 173.2)
- R2: value 10k -> 1K
- R3: value 10k -> 10K
- moved R2 9.16 mm to (55.8, 173.2), turned to 0 degrees
- moved R3 5.12 mm to (67.9, 173.2)
Connections:
- R2 pad 1: Net-(C13-Pad1) -> Net-(Q1-Pad3)
- R2 pad 2: Net-(R2-Pad2) -> Net-(BT1-Pad1)
- R3 pad 1: Net-(C13-Pad1) -> Net-(R3-Pad1)
- R3 pad 2: Net-(R3-Pad2) -> +5V
- S3 pad 1: Net-(D3-Pad1) -> /x3_WR
- S3 pad 2: Net-(R3-Pad2) -> Net-(R3-Pad1)
- U13 pad 22: Net-(R2-Pad2) -> Net-(Q1-Pad3)
- U13 pad 24: Net-(R2-Pad2) -> Net-(U11-Pad4)
- U13 pad 29: Net-(R3-Pad2) -> Net-(R3-Pad1)
- U2 pad 10: Net-(U2-Pad10) -> (no net)
- U2 pad 11: /x3_WR -> GND
- U2 pad 3: Net-(U11-Pad4) -> GND
- U2 pad 4: Net-(U2-Pad4) -> (no net)
- U2 pad 5: Net-(U2-Pad4) -> GND
- U2 pad 6: Net-(R2-Pad2) -> (no net)
- U2 pad 8: Net-(D3-Pad2) -> (no net)
- U2 pad 9: Net-(U2-Pad10) -> GND
Routing:
- net Net-(R2-Pad2): track 134.3 -> 0.00 mm
- net Net-(D3-Pad2): track 102.2 -> 0.00 mm
- net Net-(R3-Pad2): track 50.3 -> 0.00 mm
- net Net-(R3-Pad1): track 0.00 -> 47.7 mm
- net GND: track 593.4 -> 639.4 mm, vias 2 -> 1
- net Net-(U11-Pad4): track 88.5 -> 123.8 mm, vias 0 -> 1
- net +5V: track 463.7 -> 495.0 mm, vias 0 -> 1
- net /x1_WR: track 128.4 -> 157.4 mm, vias 1 -> 0
- net Net-(BT1-Pad1): track 10.8 -> 39.8 mm
- net /D3: track 124.9 -> 153.4 mm, vias 1 -> 2
- net Net-(D3-Pad1): track 25.6 -> 0.00 mm
- net Net-(U13-Pad25): track 76.1 -> 56.0 mm
- net Net-(C13-Pad1): track 43.9 -> 25.2 mm
- net Net-(U8-Pad12): track 44.3 -> 62.2 mm, vias 1 -> 2
- net /x3_WR: track 99.8 -> 83.0 mm, vias 1 -> 0
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Other:
- board text added: "1k"
- board text added: "2N7000"
- board text added: "EMM for MZ-2000 Rev1.5"
- board text removed: "1S4"
- board text removed: "EMM for MZ-2000 Rev1.2"
