File: Kicad/EMM/MZ-2000_EMM.sch (KiCad schematic (older format))
At the start: 40 parts, among them J1 Conn_02x22_Row_Letter_First, U1 74LS04, U10 74LS193, U11 74LS138, U12 74LS138, U13 HM628512LFP-5, U14 74LS11, U15 74LS245, U2 74LS04, U3 74LS14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

Commit message: Add files via upload
Parts:
- added D3: 1S4, Diode_THT:D_DO-41_SOD81_P10.16mm_Horizontal, symbol Diode:1N4001
- added R3: 10k, Resistor_THT:R_Axial_DIN0207_L6.3mm_D2.5mm_P7.62mm_Horizontal, symbol Device:R
- added S3: SLIDE_SWITCH_3P, Connector_PinHeader_2.54mm:PinHeader_1x03_P2.54mm_Vertical, symbol Memory_RAM2:SLIDE_SWITCH_3P
Connections:
- wire segments 465 -> 472
- no-connect marks 46 -> 43
Other:
- moved on the sheet: BT1, D1, D2, R2, U2B, U2C, U2D, U2E, U2F

Commit message: Add files via upload
Parts:
- D1, D2: value 1S4 -> 1N4148
Connections:
- no-connect marks 43 -> 42
Changed lines of the file:
@@
 AR Path="/692BBABE" Ref="D2"  Part="1"
 F 0 "D2" H 16250 7417 50  0000 C CNN
-F 1 "1S4" H 16250 7326 50  0000 C CNN
+F 1 "1N4148" H 16250 7326 50  0000 C CNN
 F 2 "Diode_THT:D_DO-41_SOD81_P10.16mm_Horizontal" H 16250 7025 50  0001 C CNN
 F 3 "http://www.vishay.com/docs/88503/1n4001.pdf" H 16250 7200 50  0001 C CNN
@@
 AR Path="/692BBAC9" Ref="D1"  Part="1"
 F 0 "D1" H 15250 7467 50  0000 C CNN
-F 1 "1S4" H 15250 7376 50  0000 C CNN
+F 1 "1N4148" H 15250 7376 50  0000 C CNN
 F 2 "Diode_THT:D_DO-41_SOD81_P10.16mm_Horizontal" H 15250 7075 50  0001 C CNN
 F 3 "http://www.vishay.com/docs/88503/1n4001.pdf" H 15250 7250 50  0001 C CNN
@@
 $EndComp
 Connection ~ 13100 2900
-NoConn ~ 14600 9500
 $Comp
 L 74xx:74LS04 U1
@@
 Wire Wire Line
 	14050 6300 14450 6300
+Wire Wire Line
+	15050 5700 14750 5700
+Wire Wire Line
+	14750 5700 14750 4100
+Connection ~ 14750 4100
+Wire Wire Line
+	14750 4100 15400 4100
+Wire Wire Line
+	15650 5700 15950 5700
+Wire Wire Line
+	16550 5700 16650 5700
+Wire Wire Line
+	17850 6050 17850 7800
+Wire Wire Line
+	16100 10100 17850 10100
+Wire Wire Line
+	17600 7800 17850 7800
+Connection ~ 17850 7800
+Wire Wire Line
+	17850 7800 17850 10100
+Wire Wire Line
+	17300 7800 15600 7800
+Connection ~ 15600 7800
+Wire Wire Line
+	15600 7800 15600 8150
+$Comp
+L Memory_RAM2:SLIDE_SWITCH_3P S3
+U 1 1 696442FF
+P 17350 5500
+F 0 "S3" H 17350 5565 50  0000 C CNN
+F 1 "SLIDE_SWITCH_3P" H 17350 5474 50  0000 C CNN
+F 2 "Connector_PinHeader_2.54mm:PinHeader_1x03_P2.54mm_Vertical" H 17350 5525 50  0001 C CNN
+F 3 "" H 17350 5525 50  0001 C CNN
+	1    17350 5500
+	1    0    0    -1
+$EndComp
+Wire Wire Line
+	16950 5700 17150 5700
+Wire Wire Line
+	17850 6050 17350 6050
+Wire Wire Line
+	17350 6050 17350 5850
+NoConn ~ 17550 5700
+Wire Wire Line
+	15050 6300 17700 6300
+Wire Wire Line
+	4600 15700 4600 15050
+Connection ~ 4600 15700
+Connection ~ 4600 15050
 $Comp
 L Diode:1N4001 D?
@@
 	-1   0    0    -1
 $EndComp
-Wire Wire Line
-	15050 5700 14750 5700
-Wire Wire Line
-	14750 5700 14750 4100
-Connection ~ 14750 4100
-Wire Wire Line
-	14750 4100 15400 4100
-Wire Wire Line
-	15650 5700 15950 5700
-Wire Wire Line
-	16550 5700 16650 5700
-Wire Wire Line
-	17850 6050 17850 7800
-Wire Wire Line
-	16100 10100 17850 10100
-Wire Wire Line
-	17600 7800 17850 7800
-Connection ~ 17850 7800
-Wire Wire Line
-	17850 7800 17850 10100
-Wire Wire Line
-	17300 7800 15600 7800
-Connection ~ 15600 7800
-Wire Wire Line
-	15600 7800 15600 8150
-$Comp
-L Memory_RAM2:SLIDE_SWITCH_3P S3
-U 1 1 696442FF
-P 17350 5500
-F 0 "S3" H 17350 5565 50  0000 C CNN
-F 1 "SLIDE_SWITCH_3P" H 17350 5474 50  0000 C CNN
-F 2 "Connector_PinHeader_2.54mm:PinHeader_1x03_P2.54mm_Vertical" H 17350 5525 50  0001 C CNN
-F 3 "" H 17350 5525 50  0001 C CNN
-	1    17350 5500
-	1    0    0    -1
-$EndComp
-Wire Wire Line
-	16950 5700 17150 5700
-Wire Wire Line
-	17850 6050 17350 6050
-Wire Wire Line
-	17350 6050 17350 5850
-NoConn ~ 17550 5700
-Wire Wire Line
-	15050 6300 17700 6300
-Wire Wire Line
-	4600 15700 4600 15050
-Connection ~ 4600 15700
-Connection ~ 4600 15050
 $EndSCHEMATC

Commit message: Add files via upload
Parts:
- removed D3: 1S4, Diode_THT:D_DO-41_SOD81_P10.16mm_Horizontal, symbol Diode:1N4001
- added Q1: 2N7000, Package_TO_SOT_THT:TO-92, symbol Device:Q_NMOS_SGD
- R2: value 10k -> 1K
- R3: value 10k -> 10K
Connections:
- wire segments 472 -> 479
- no-connect marks 42 -> 46
Other:
- moved on the sheet: U2B, U2C, U2D, U2E
