File: Kicad/EMM&CMU/MZ-2000_EMM_CMU.kicad_pcb (KiCad board)
At the start: 2 copper layers, 115.8 x 158.4 mm, 45 parts, among them J1 Conn_02x22_Row_Letter_First, J2 Conn_02x25_Odd_Even, U1 74LS04, U10 74LS193, U11 74LS138, U12 74LS138, U13 HM628512LFP-5, U14 74LS11, U15 74LS245, U2 74LS04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

Commit message: Add files via upload
Parts:
- added D3: 1S4, Diode_THT:D_DO-41_SOD81_P10.16mm_Horizontal, F.Cu at (58.3, 177.6)
- added R3: 10k, Resistor_THT:R_Axial_DIN0207_L6.3mm_D2.5mm_P7.62mm_Horizontal, F.Cu at (69.2, 169.0)
- added S3: SLIDE_SWITCH_3P, Connector_PinHeader_2.54mm:PinHeader_1x03_P2.54mm_Vertical, F.Cu at (84.3, 192.4)
- moved BT1 2.24 mm to (104.2, 174.8)
- moved D1 2.18 mm to (81.2, 177.9)
- moved R2 2.11 mm to (65.4, 169.0)
- moved D2 0.91 mm to (81.2, 169.0)
Connections:
- U11 pad 4: Net-(R2-Pad2) -> Net-(U11-Pad4)
- U11 pad 5: Net-(R2-Pad2) -> Net-(U11-Pad4)
- U12 pad 4: Net-(R2-Pad2) -> Net-(U11-Pad4)
- U12 pad 5: Net-(R2-Pad2) -> Net-(U11-Pad4)
- U13 pad 29: /x3_WR -> Net-(R3-Pad2)
- U2 pad 10: (no net) -> Net-(U2-Pad10)
- U2 pad 11: GND -> /x3_WR
- U2 pad 3: GND -> Net-(U11-Pad4)
- U2 pad 4: (no net) -> Net-(U2-Pad4)
- U2 pad 5: GND -> Net-(U2-Pad4)
- U2 pad 6: (no net) -> Net-(R2-Pad2)
- U2 pad 8: (no net) -> Net-(D3-Pad2)
- U2 pad 9: GND -> Net-(U2-Pad10)
- U5 pad 8: Net-(R2-Pad2) -> Net-(U11-Pad4)
Routing:
- net Net-(D3-Pad2): track 0.00 -> 111.9 mm
- net Net-(U11-Pad4): track 0.00 -> 88.2 mm
- net Net-(R3-Pad2): track 0.00 -> 37.5 mm
- net Net-(D3-Pad1): track 0.00 -> 32.1 mm
- net Net-(U13-Pad25): track 60.7 -> 76.1 mm, vias 1 -> 0
- net /A7: track 213.2 -> 228.2 mm, vias 1 -> 3
- net /D4: track 201.2 -> 213.8 mm, vias 2 -> 3
- net /A4: track 173.2 -> 185.3 mm
- net GND: track 695.6 -> 684.7 mm, vias 3 -> 2
- net /x3_WR: track 91.4 -> 102.2 mm, vias 0 -> 1
- net Net-(U13-Pad8): track 35.0 -> 45.4 mm, vias 1 -> 0
- net /~WR: track 215.6 -> 225.0 mm
- net /D7: track 221.1 -> 229.5 mm, vias 1 -> 2
- net /D5: track 207.0 -> 215.1 mm
- net /A2: track 190.3 -> 197.9 mm, vias 2 -> 0
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Other:
- board text added: "EMM & CMU-800 for MZ-2000 Rev1.2"
- board text added: "RAM"
- board text added: "ROM"
- board text removed: "EMM & CMU-800 for MZ-2000"

Commit message: Add files via upload
Parts:
- D1, D2: value 1S4 -> 1N4148
Other:
- board text added: "1N4148"

Commit message: Add files via upload
Parts:
- removed D3: 1S4, Diode_THT:D_DO-41_SOD81_P10.16mm_Horizontal
- added Q1: 2N7000, Package_TO_SOT_THT:TO-92, F.Cu at (49.7, 145.9)
- R2: value 10k -> 1k
- R3: value 10k -> 100
- moved C13 29.0 mm to (86.0, 125.7)
- moved U10 29.0 mm to (100.0, 99.7)
- moved U12 29.0 mm to (140.0, 99.7)
- moved BT1 29.0 mm to (105.2, 145.8)
- moved C1 29.0 mm to (112.1, 57.2)
- moved C10 29.0 mm to (103.2, 104.8)
- moved C11 29.0 mm to (143.2, 89.6)
- moved C12 29.0 mm to (143.2, 104.8)
- moved C14 29.0 mm to (140.6, 121.9)
- moved C15 29.0 mm to (117.2, 121.9)
- moved C16 29.0 mm to (46.7, 64.2)
- moved C2 29.0 mm to (87.3, 57.2)
- moved C3 29.0 mm to (62.5, 57.2)
- moved C4 29.0 mm to (70.2, 76.9)
- moved C5 29.0 mm to (140.0, 73.7)
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Connections:
- R2 pad 1: Net-(C13-Pad1) -> Net-(Q1-Pad3)
- R2 pad 2: Net-(R2-Pad2) -> Net-(BT1-Pad1)
- R3 pad 1: Net-(C13-Pad1) -> Net-(R3-Pad1)
- R3 pad 2: Net-(R3-Pad2) -> +5V
- S3 pad 1: Net-(D3-Pad1) -> /x3_WR
- S3 pad 2: Net-(R3-Pad2) -> Net-(R3-Pad1)
- U13 pad 22: Net-(R2-Pad2) -> Net-(Q1-Pad3)
- U13 pad 24: Net-(R2-Pad2) -> Net-(U11-Pad4)
- U13 pad 29: Net-(R3-Pad2) -> Net-(R3-Pad1)
- U2 pad 10: Net-(U2-Pad10) -> (no net)
- U2 pad 11: /x3_WR -> GND
- U2 pad 3: Net-(U11-Pad4) -> GND
- U2 pad 4: Net-(U2-Pad4) -> (no net)
- U2 pad 5: Net-(U2-Pad4) -> GND
- U2 pad 6: Net-(R2-Pad2) -> (no net)
- U2 pad 8: Net-(D3-Pad2) -> (no net)
- U2 pad 9: Net-(U2-Pad10) -> GND
Routing:
- net Net-(R2-Pad2): track 148.8 -> 0.00 mm, vias 1 -> 0
- net Net-(D3-Pad2): track 111.9 -> 0.00 mm
- net +5V: track 453.3 -> 514.6 mm
- net Net-(U11-Pad4): track 88.2 -> 148.5 mm
- net Net-(R3-Pad2): track 37.5 -> 0.00 mm
- net Net-(R3-Pad1): track 0.00 -> 36.8 mm
- net Net-(D3-Pad1): track 32.1 -> 0.00 mm
- net Net-(BT1-Pad1): track 14.1 -> 43.3 mm
- net /A4: track 185.3 -> 157.2 mm, vias 1 -> 2
- net /D7: track 229.5 -> 209.5 mm
- net Net-(Q1-Pad3): track 0.00 -> 18.3 mm
- net Net-(U13-Pad25): track 76.1 -> 58.6 mm, vias 0 -> 1
- net Net-(C13-Pad1): track 41.8 -> 24.7 mm
- net /x3_WR: track 102.2 -> 86.1 mm, vias 1 -> 0
- net /A6: track 164.7 -> 179.4 mm, vias 1 -> 3
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Other:
- board text added: "1k"
- board text added: "2N7000"
- board text added: "EMM & CMU-800 for MZ-2000 Rev1.5"
- board text removed: "1S4"
- board text removed: "EMM & CMU-800 for MZ-2000 Rev1.2"
