File: Kicad/EMM&CMU/MZ-2000_EMM_CMU.sch (KiCad schematic (older format))
At the start: 41 parts, among them J1 Conn_02x22_Row_Letter_First, J2 Conn_02x25_Odd_Even, U1 74LS04, U10 74LS193, U11 74LS138, U12 74LS138, U13 HM628512LFP-5, U14 74LS11, U15 74LS245, U2 74LS04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

Commit message: Add files via upload
Parts:
- added D3: 1S4, Diode_THT:D_DO-41_SOD81_P10.16mm_Horizontal, symbol Diode:1N4001
- added R3: 10k, Resistor_THT:R_Axial_DIN0207_L6.3mm_D2.5mm_P7.62mm_Horizontal, symbol Device:R
- added S3: SLIDE_SWITCH_3P, Connector_PinHeader_2.54mm:PinHeader_1x03_P2.54mm_Vertical, symbol Memory_RAM2:SLIDE_SWITCH_3P
Connections:
- wire segments 485 -> 492
- no-connect marks 76 -> 73
Other:
- moved on the sheet: BT1, D1, D2, R2, U2B, U2C, U2D, U2E, U2F

Commit message: Add files via upload
Parts:
- D1, D2: value 1S4 -> 1N4148
Connections:
- no-connect marks 73 -> 72
Changed lines of the file:
@@
 AR Path="/692BBABE" Ref="D2"  Part="1"
 F 0 "D2" H 16250 7867 50  0000 C CNN
-F 1 "1S4" H 16250 7776 50  0000 C CNN
+F 1 "1N4148" H 16250 7776 50  0000 C CNN
 F 2 "Diode_THT:D_DO-41_SOD81_P10.16mm_Horizontal" H 16250 7475 50  0001 C CNN
 F 3 "http://www.vishay.com/docs/88503/1n4001.pdf" H 16250 7650 50  0001 C CNN
@@
 AR Path="/692BBAC9" Ref="D1"  Part="1"
 F 0 "D1" H 15250 7917 50  0000 C CNN
-F 1 "1S4" H 15250 7826 50  0000 C CNN
+F 1 "1N4148" H 15250 7826 50  0000 C CNN
 F 2 "Diode_THT:D_DO-41_SOD81_P10.16mm_Horizontal" H 15250 7525 50  0001 C CNN
 F 3 "http://www.vishay.com/docs/88503/1n4001.pdf" H 15250 7700 50  0001 C CNN
@@
 Connection ~ 13100 2900
 NoConn ~ 5300 3300
-NoConn ~ 14600 9500
 $Comp
 L 74xx:74LS04 U1

Commit message: Add files via upload
Parts:
- removed D3: 1S4, Diode_THT:D_DO-41_SOD81_P10.16mm_Horizontal, symbol Diode:1N4001
- added Q1: 2N7000, Package_TO_SOT_THT:TO-92, symbol Device:Q_NMOS_SGD
- R2: value 10k -> 1k
- R3: value 10k -> 100
Connections:
- wire segments 492 -> 497
- no-connect marks 72 -> 76
Other:
- moved on the sheet: BT1, D1, D2, U2B, U2C, U2D, U2E
